Commit message: Cupboard URDF with three drawers working

File: data/cupboard_drawers/cupboard_drawers.urdf (robot description, URDF)
Before this commit: robot cupboard_drawers, 6 links, 5 joints
Links:
- removed link fr_back_wall
- removed link fr_bottom_wall
- removed link fr_left_wall
- removed link fr_right_wall
- removed link fr_top_wall
- added link drawer1_back_wall, mass 0.2; collision box size=1.34 0.025 0.895; visual box size=1.34 0.025 0.895
- added link drawer1_bottom_wall, mass 0.2; collision box size=1.39 0.025 0.46; visual box size=1.39 0.025 0.46
- added link drawer1_left_wall, mass 0.2; collision box size=0.46 0.025 0.895; visual box size=0.46 0.025 0.895
- added link drawer1_right_wall, mass 0.2; collision box size=0.46 0.025 0.895; visual box size=0.46 0.025 0.895
- added link drawer1_top_wall, mass 0.2; collision box size=1.39 0.025 0.46; visual box size=1.39 0.025 0.46
- added link frame_back_wall, mass 0.2; collision box size=1.4 0.05 1.4; visual box size=1.4 0.05 1.4
- added link frame_bottom_wall, mass 0.2; collision box size=1.5 0.05 1.0; visual box size=1.5 0.05 1.0
- added link frame_left_wall, mass 0.2; collision box size=1.0 0.05 1.4; visual box size=1.0 0.05 1.4
- added link frame_right_wall, mass 0.2; collision box size=1.0 0.05 1.4; visual box size=1.0 0.05 1.4
- added link frame_top_wall, mass 0.2; collision box size=1.5 0.05 1.0; visual box size=1.5 0.05 1.0
Joints:
- removed joint fr_back_joint
- removed joint fr_bottom_joint
- removed joint fr_left_joint
- removed joint fr_right_joint
- removed joint fr_top_joint
- added joint drawer1_bottom_joint: type fixed, parent drawer1_back_wall, child drawer1_bottom_wall, origin xyz=0 -0.2175 -0.46 rpy=1.57079632679 0 0
- added joint drawer1_joint: type prismatic, parent base_link, child drawer1_back_wall, origin xyz=0 -0.0275 1.7 rpy=-1.57079632679 0 0, axis 0 0 -1, limit lower=-10.0 upper=10.5 effort=1.0 velocity=1.5
- added joint drawer1_left_joint: type fixed, parent drawer1_back_wall, child drawer1_left_wall, origin xyz=-0.6825 -0.2175 0 rpy=0 0 1.57079632679
- added joint drawer1_right_joint: type fixed, parent drawer1_back_wall, child drawer1_right_wall, origin xyz=0.6825 -0.2175 0 rpy=0 0 1.57079632679
- added joint drawer1_top_joint: type fixed, parent drawer1_back_wall, child drawer1_top_wall, origin xyz=0 -0.2175 0.46 rpy=1.57079632679 0 0
- added joint frame_bottom_joint: type fixed, parent frame_back_wall, child frame_bottom_wall, origin xyz=0 -0.475 -0.725 rpy=1.57079632679 0 0
- added joint frame_joint: type fixed, parent base_link, child frame_back_wall, origin xyz=0 0.475 0.75 rpy=0 0 0
- added joint frame_left_joint: type fixed, parent frame_back_wall, child frame_left_wall, origin xyz=-0.725 -0.475 0 rpy=0 0 1.57079632679
- added joint frame_right_joint: type fixed, parent frame_back_wall, child frame_right_wall, origin xyz=0.725 -0.475 0 rpy=0 0 1.57079632679
- added joint frame_top_joint: type fixed, parent frame_back_wall, child frame_top_wall, origin xyz=0 -0.475 0.725 rpy=1.57079632679 0 0

File: data/cupboard_drawers/cupboard_drawers.urdf.xacro (robot description, xacro)
@@ -13,5 +13,5 @@
   </geometry>
 </xacro:macro>
-<xacro:macro name="wall" params="prefix width height">
+<xacro:macro name="wall" params="prefix width height thickness">
   <link name="${prefix}_wall">
     <contact>
@@ -20,9 +20,9 @@
     <inertial>
       <origin rpy="0 0 0" xyz="0 0 0"/>
-       <mass value=".2"/>
+       <mass value="0.2"/>
        <inertia ixx="1" ixy="0" ixz="0" iyy="1" iyz="0" izz="1"/>
     </inertial>
     <visual>
-      <xacro:ori_geo width="${width}" depth="${wall_thickness}" height="${height}"/>
+      <xacro:ori_geo width="${width}" depth="${thickness}" height="${height}"/>
       <material name="white">
         <color rgba="1 1 1 1"/>
@@ -30,38 +30,73 @@
     </visual>
     <collision>
-      <xacro:ori_geo width="${width}" depth="${wall_thickness}" height="${height}"/>
+      <xacro:ori_geo width="${width}" depth="${thickness}" height="${height}"/>
     </collision>
   </link>
 </xacro:macro>
+<xacro:macro name="corpus" params="prefix width depth height wall_thickness">
+  <xacro:wall prefix="${prefix}_back" width="${width-2*wall_thickness}" height="${height-2*wall_thickness}" thickness="${wall_thickness}"/>
+  <xacro:wall prefix="${prefix}_bottom" width="${width}" height="${depth}" thickness="${wall_thickness}"/>
+  <joint name="${prefix}_bottom_joint" type="fixed">
+    <origin xyz="0 -${depth/2-wall_thickness/2} -${height/2-wall_thickness/2}" rpy="${pi/2} 0 0"/>
+    <parent link="${prefix}_back_wall"/>
+    <child link="${prefix}_bottom_wall"/>
+  </joint>
+  <xacro:wall prefix="${prefix}_left" width="${depth}" height="${height-2*wall_thickness}" thickness="${wall_thickness}"/>
+  <joint name="${prefix}_left_joint" type="fixed">
+    <origin xyz="-${width/2-wall_thickness/2} -${depth/2-wall_thickness/2} 0" rpy="0 0 ${pi/2}"/>
+    <parent link="${prefix}_back_wall"/>
+    <child link="${prefix}_left_wall"/>
+  </joint>
+  <xacro:wall prefix="${prefix}_right" width="${depth}" height="${height-2*wall_thickness}" thickness="${wall_thickness}"/>
+  <joint name="${prefix}_right_joint" type="fixed">
+    <origin xyz="${width/2-wall_thickness/2} -${depth/2-wall_thickness/2} 0" rpy="0 0 ${pi/2}"/>
+    <parent link="${prefix}_back_wall"/>
+    <child link="${prefix}_right_wall"/>
+  </joint>
+  <xacro:wall prefix="${prefix}_top" width="${width}" height="${depth}" thickness="${wall_thickness}"/>
+  <joint name="${prefix}_top_joint" type="fixed">
+    <origin xyz="0 -${depth/2-wall_thickness/2} ${height/2-wall_thickness/2}" rpy="${pi/2} 0 0"/>
+    <parent link="${prefix}_back_wall"/>
+    <child link="${prefix}_top_wall"/>
+  </joint>
+</xacro:macro>
+<xacro:macro name="drawer" params="index">
+  <xacro:property name="drawer_height" value="${(total_height-2*wall_thickness-(num_drawers+1)*drawer_spacing)/num_drawers}"/>
+  <xacro:corpus prefix="drawer${index}"
+              width="${total_width-2*(wall_thickness+drawer_spacing)}"
+              depth="${drawer_height}"
+              height="${total_depth-wall_thickness-drawer_spacing}"
+              wall_thickness="${wall_thickness*0.5}"/>
+  <joint name="drawer${index}_joint" type="prismatic">
+    <origin xyz="0 -${(wall_thickness+drawer_spacing)/2} ${wall_thickness+drawer_spacing+0.5*0.5*wall_thickness + (index-1)*(drawer_height+drawer_spacing)}" rpy="-${pi/2} 0 0"/>
+    <parent link="base_link"/>
+    <child link="drawer${index}_back_wall"/>
+    <axis xyz="0 -1 0"/>
+    <dynamics damping="0.1"/>
+    <limit lower="0.0" upper="1.5" effort="0.0" velocity="0.5"/>
+  </joint>
+</xacro:macro>
 <link name="base_link"/>
-<xacro:wall prefix="fr_bottom" width="${total_width}" height="${total_depth}"/>
-<joint name="fr_bottom_joint" type="fixed">
-  <origin xyz="0 0 ${wall_thickness/2}" rpy="${pi/2} 0 0"/>
-  <parent link="base_link"/>
-  <child link="fr_bottom_wall"/>
-</joint>
-<xacro:wall prefix="fr_back" width="${total_width-2*wall_thickness}" height="${total_height-2*wall_thickness}"/>
-<joint name="fr_back_joint" type="fixed">
+<xacro:corpus prefix="frame" width="${total_width}" depth="${total_depth}" height="${total_height}" wall_thickness="${wall_thickness}"/>
+<joint name="frame_joint" type="fixed">
   <origin xyz="0 ${total_depth/2-wall_thickness/2} ${total_height/2}" rpy="0 0 0"/>
   <parent link="base_link"/>
-  <child link="fr_back_wall"/>
+  <child link="frame_back_wall"/>
 </joint>
-<xacro:wall prefix="fr_left" width="${total_depth}" height="${total_height-2*wall_thickness}"/>
-<joint name="fr_left_joint" type="fixed">
-  <origin xyz="-${total_width/2-wall_thickness/2} 0 ${total_height/2}" rpy="0 0 ${pi/2}"/>
+<!-- <xacro:drawer index="1"/>
+<xacro:drawer index="2"/>
+<xacro:drawer index="3"/> -->
+<xacro:corpus prefix="drawer1"
+              width="${total_width-2*(wall_thickness+drawer_spacing)}"
+              depth="${(total_height-2*wall_thickness-(num_drawers+1)*drawer_spacing)/num_drawers}"
+              height="${total_depth-wall_thickness-drawer_spacing}"
+              wall_thickness="${wall_thickness*0.5}"/>
+<joint name="drawer1_joint" type="prismatic">
+  <origin xyz="0 -${(wall_thickness+drawer_spacing)/2} ${1.7}" rpy="-${pi/2} 0 0"/>
   <parent link="base_link"/>
-  <child link="fr_left_wall"/>
-</joint>
-<xacro:wall prefix="fr_right" width="${total_depth}" height="${total_height-2*wall_thickness}"/>
-<joint name="fr_right_joint" type="fixed">
-  <origin xyz="${total_width/2-wall_thickness/2} 0 ${total_height/2}" rpy="0 0 ${pi/2}"/>
-  <parent link="base_link"/>
-  <child link="fr_right_wall"/>
-</joint>
-<xacro:wall prefix="fr_top" width="${total_width}" height="${total_depth}"/>
-<joint name="fr_top_joint" type="fixed">
-  <origin xyz="0 0 ${total_height-wall_thickness/2}" rpy="${pi/2} 0 0"/>
-  <parent link="base_link"/>
-  <child link="fr_top_wall"/>
+  <child link="drawer1_back_wall"/>
+  <axis xyz="0 0 -1"/>
+  <dynamics damping="0.0"/>
+  <limit lower="-10.0" upper="10.5" effort="1.0" velocity="1.5"/>
 </joint>
 </robot>

Commit message: Cupboard working with joint limits and damping

File: data/cupboard_drawers/cupboard_drawers.urdf (robot description, URDF)
Before this commit: robot cupboard_drawers, 11 links, 10 joints
Links:
- added link drawer1_handle, mass 0.2; collision cylinder length=0.3 radius=0.03; visual cylinder length=0.3 radius=0.03
- added link drawer2_back_wall, mass 0.2; collision box size=1.34 0.025 0.895; visual box size=1.34 0.025 0.895
- added link drawer2_bottom_wall, mass 0.2; collision box size=1.39 0.025 0.46; visual box size=1.39 0.025 0.46
- added link drawer2_handle, mass 0.2; collision cylinder length=0.3 radius=0.03; visual cylinder length=0.3 radius=0.03
- added link drawer2_left_wall, mass 0.2; collision box size=0.46 0.025 0.895; visual box size=0.46 0.025 0.895
- added link drawer2_right_wall, mass 0.2; collision box size=0.46 0.025 0.895; visual box size=0.46 0.025 0.895
- added link drawer2_top_wall, mass 0.2; collision box size=1.39 0.025 0.46; visual box size=1.39 0.025 0.46
- added link drawer3_back_wall, mass 0.2; collision box size=1.34 0.025 0.895; visual box size=1.34 0.025 0.895
- added link drawer3_bottom_wall, mass 0.2; collision box size=1.39 0.025 0.46; visual box size=1.39 0.025 0.46
- added link drawer3_handle, mass 0.2; collision cylinder length=0.3 radius=0.03; visual cylinder length=0.3 radius=0.03
- added link drawer3_left_wall, mass 0.2; collision box size=0.46 0.025 0.895; visual box size=0.46 0.025 0.895
- added link drawer3_right_wall, mass 0.2; collision box size=0.46 0.025 0.895; visual box size=0.46 0.025 0.895
- added link drawer3_top_wall, mass 0.2; collision box size=1.39 0.025 0.46; visual box size=1.39 0.025 0.46
- link base_link: mass None -> 0.0
Joints:
- removed joint drawer1_joint
- added joint drawer1_handle_joint: type fixed, parent drawer1_back_wall, child drawer1_handle, origin xyz=0 -0.23 -0.52 rpy=0 1.57079632679 0
- added joint drawer2_bottom_joint: type fixed, parent drawer2_back_wall, child drawer2_bottom_wall, origin xyz=0 -0.2175 -0.46 rpy=1.57079632679 0 0
- added joint drawer2_handle_joint: type fixed, parent drawer2_back_wall, child drawer2_handle, origin xyz=0 -0.23 -0.52 rpy=0 1.57079632679 0
- added joint drawer2_left_joint: type fixed, parent drawer2_back_wall, child drawer2_left_wall, origin xyz=-0.6825 -0.2175 0 rpy=0 0 1.57079632679
- added joint drawer2_right_joint: type fixed, parent drawer2_back_wall, child drawer2_right_wall, origin xyz=0.6825 -0.2175 0 rpy=0 0 1.57079632679
- added joint drawer2_top_joint: type fixed, parent drawer2_back_wall, child drawer2_top_wall, origin xyz=0 -0.2175 0.46 rpy=1.57079632679 0 0
- added joint drawer3_bottom_joint: type fixed, parent drawer3_back_wall, child drawer3_bottom_wall, origin xyz=0 -0.2175 -0.46 rpy=1.57079632679 0 0
- added joint drawer3_handle_joint: type fixed, parent drawer3_back_wall, child drawer3_handle, origin xyz=0 -0.23 -0.52 rpy=0 1.57079632679 0
- added joint drawer3_left_joint: type fixed, parent drawer3_back_wall, child drawer3_left_wall, origin xyz=-0.6825 -0.2175 0 rpy=0 0 1.57079632679
- added joint drawer3_right_joint: type fixed, parent drawer3_back_wall, child drawer3_right_wall, origin xyz=0.6825 -0.2175 0 rpy=0 0 1.57079632679
- added joint drawer3_top_joint: type fixed, parent drawer3_back_wall, child drawer3_top_wall, origin xyz=0 -0.2175 0.46 rpy=1.57079632679 0 0
- added joint drawer_joint1: type prismatic, parent base_link, child drawer1_back_wall, origin xyz=0 -0.0275 0.0675 rpy=-1.57079632679 0 0, axis 0 0 -1, limit lower=0.0 upper=0.8 effort=10.0 velocity=1.5
- added joint drawer_joint2: type prismatic, parent base_link, child drawer2_back_wall, origin xyz=0 -0.0275 0.5325 rpy=-1.57079632679 0 0, axis 0 0 -1, limit lower=0.0 upper=0.8 effort=10.0 velocity=1.5
- added joint drawer_joint3: type prismatic, parent base_link, child drawer3_back_wall, origin xyz=0 -0.0275 0.9975 rpy=-1.57079632679 0 0, axis 0 0 -1, limit lower=0.0 upper=0.8 effort=10.0 velocity=1.5

File: data/cupboard_drawers/cupboard_drawers.urdf.xacro (robot description, xacro)
@@ -68,14 +68,47 @@
               height="${total_depth-wall_thickness-drawer_spacing}"
               wall_thickness="${wall_thickness*0.5}"/>
-  <joint name="drawer${index}_joint" type="prismatic">
+  <joint name="drawer_joint${index}" type="prismatic">
     <origin xyz="0 -${(wall_thickness+drawer_spacing)/2} ${wall_thickness+drawer_spacing+0.5*0.5*wall_thickness + (index-1)*(drawer_height+drawer_spacing)}" rpy="-${pi/2} 0 0"/>
     <parent link="base_link"/>
     <child link="drawer${index}_back_wall"/>
-    <axis xyz="0 -1 0"/>
-    <dynamics damping="0.1"/>
-    <limit lower="0.0" upper="1.5" effort="0.0" velocity="0.5"/>
+    <axis xyz="0 0 -1"/>
+    <dynamics damping="8.0"/>
+    <limit lower="0.0" upper="${0.8*total_depth}" effort="10.0" velocity="1.5"/>
+  </joint>
+  <link name="drawer${index}_handle">
+    <inertial>
+      <origin rpy="0 0 0" xyz="0 0 0"/>
+      <mass value="0.2"/>
+      <inertia ixx="1" ixy="0" ixz="0" iyy="1" iyz="0" izz="1"/>
+    </inertial>
+    <collision>
+      <origin rpy="0 0 0" xyz="0 0 0"/>
+      <geometry>
+        <cylinder radius="0.03" length="0.3"/>
+      </geometry>
+    </collision>
+    <visual>
+      <origin rpy="0 0 0" xyz="0 0 0"/>
+      <geometry>
+        <cylinder radius="0.03" length="0.3"/>
+      </geometry>
+      <material name="white">
+        <color rgba="1 1 1 1"/>
+      </material>
+    </visual>
+  </link>
+  <joint name="drawer${index}_handle_joint" type="fixed">
+    <origin xyz="0 ${-drawer_height/2} ${-total_depth/2-0.02}" rpy="0 ${pi/2} 0"/>
+    <parent link="drawer${index}_back_wall"/>
+    <child link="drawer${index}_handle"/>
   </joint>
 </xacro:macro>
-<link name="base_link"/>
+<link name="base_link">
+  <inertial>
+    <origin rpy="0 0 0" xyz="0 0 0"/>
+    <mass value="0.0"/>
+    <inertia ixx="1" ixy="0" ixz="0" iyy="1" iyz="0" izz="1"/>
+  </inertial>
+</link>
 <xacro:corpus prefix="frame" width="${total_width}" depth="${total_depth}" height="${total_height}" wall_thickness="${wall_thickness}"/>
 <joint name="frame_joint" type="fixed">
@@ -84,19 +117,6 @@
   <child link="frame_back_wall"/>
 </joint>
-<!-- <xacro:drawer index="1"/>
+<xacro:drawer index="1"/>
 <xacro:drawer index="2"/>
-<xacro:drawer index="3"/> -->
-<xacro:corpus prefix="drawer1"
-              width="${total_width-2*(wall_thickness+drawer_spacing)}"
-              depth="${(total_height-2*wall_thickness-(num_drawers+1)*drawer_spacing)/num_drawers}"
-              height="${total_depth-wall_thickness-drawer_spacing}"
-              wall_thickness="${wall_thickness*0.5}"/>
-<joint name="drawer1_joint" type="prismatic">
-  <origin xyz="0 -${(wall_thickness+drawer_spacing)/2} ${1.7}" rpy="-${pi/2} 0 0"/>
-  <parent link="base_link"/>
-  <child link="drawer1_back_wall"/>
-  <axis xyz="0 0 -1"/>
-  <dynamics damping="0.0"/>
-  <limit lower="-10.0" upper="10.5" effort="1.0" velocity="1.5"/>
-</joint>
+<xacro:drawer index="3"/>
 </robot>
