Commit message: Embedded cupboard into remaining infrastructure. Changed color and size.

File: data/cupboard_drawers/cupboard_drawers.urdf (robot description, URDF)
Before this commit: robot cupboard_drawers, 24 links, 23 joints
Links:
- link drawer1_back_wall: geometry collision box size=0.8 0.015 0.535; visual box size=0.8 0.015 0.535
- link drawer1_bottom_wall: geometry collision box size=0.83 0.015 0.306666666667; visual box size=0.83 0.015 0.306666666667
- link drawer1_handle: geometry collision cylinder length=0.45 radius=0.02; visual cylinder length=0.45 radius=0.02
- link drawer1_left_wall: geometry collision box size=0.306666666667 0.015 0.535; visual box size=0.306666666667 0.015 0.535
- link drawer1_right_wall: geometry collision box size=0.306666666667 0.015 0.535; visual box size=0.306666666667 0.015 0.535
- link drawer1_top_wall: geometry collision box size=0.83 0.015 0.306666666667; visual box size=0.83 0.015 0.306666666667
- link drawer2_back_wall: geometry collision box size=0.8 0.015 0.535; visual box size=0.8 0.015 0.535
- link drawer2_bottom_wall: geometry collision box size=0.83 0.015 0.306666666667; visual box size=0.83 0.015 0.306666666667
- link drawer2_handle: geometry collision cylinder length=0.45 radius=0.02; visual cylinder length=0.45 radius=0.02
- link drawer2_left_wall: geometry collision box size=0.306666666667 0.015 0.535; visual box size=0.306666666667 0.015 0.535
- link drawer2_right_wall: geometry collision box size=0.306666666667 0.015 0.535; visual box size=0.306666666667 0.015 0.535
- link drawer2_top_wall: geometry collision box size=0.83 0.015 0.306666666667; visual box size=0.83 0.015 0.306666666667
- link drawer3_back_wall: geometry collision box size=0.8 0.015 0.535; visual box size=0.8 0.015 0.535
- link drawer3_bottom_wall: geometry collision box size=0.83 0.015 0.306666666667; visual box size=0.83 0.015 0.306666666667
- link drawer3_handle: geometry collision cylinder length=0.45 radius=0.02; visual cylinder length=0.45 radius=0.02
- link drawer3_left_wall: geometry collision box size=0.306666666667 0.015 0.535; visual box size=0.306666666667 0.015 0.535
- link drawer3_right_wall: geometry collision box size=0.306666666667 0.015 0.535; visual box size=0.306666666667 0.015 0.535
- link drawer3_top_wall: geometry collision box size=0.83 0.015 0.306666666667; visual box size=0.83 0.015 0.306666666667
- link frame_back_wall: geometry collision box size=0.84 0.03 0.94; visual box size=0.84 0.03 0.94
- link frame_bottom_wall: geometry collision box size=0.9 0.03 0.6; visual box size=0.9 0.03 0.6
- link frame_left_wall: geometry collision box size=0.6 0.03 0.94; visual box size=0.6 0.03 0.94
- link frame_right_wall: geometry collision box size=0.6 0.03 0.94; visual box size=0.6 0.03 0.94
- link frame_top_wall: geometry collision box size=0.9 0.03 0.6; visual box size=0.9 0.03 0.6
Joints:
- joint drawer1_bottom_joint: origin xyz=0 -0.2175 -0.46 rpy=1.57079632679 0 0 -> xyz=0 -0.145833333333 -0.275 rpy=1.57079632679 0 0
- joint drawer1_handle_joint: origin xyz=0 -0.23 -0.52 rpy=0 1.57079632679 0 -> xyz=0 -0.153333333333 -0.32 rpy=0 1.57079632679 0
- joint drawer1_left_joint: origin xyz=-0.6825 -0.2175 0 rpy=0 0 1.57079632679 -> xyz=-0.4075 -0.145833333333 0 rpy=0 0 1.57079632679
- joint drawer1_right_joint: origin xyz=0.6825 -0.2175 0 rpy=0 0 1.57079632679 -> xyz=0.4075 -0.145833333333 0 rpy=0 0 1.57079632679
- joint drawer1_top_joint: origin xyz=0 -0.2175 0.46 rpy=1.57079632679 0 0 -> xyz=0 -0.145833333333 0.275 rpy=1.57079632679 0 0
- joint drawer2_bottom_joint: origin xyz=0 -0.2175 -0.46 rpy=1.57079632679 0 0 -> xyz=0 -0.145833333333 -0.275 rpy=1.57079632679 0 0
- joint drawer2_handle_joint: origin xyz=0 -0.23 -0.52 rpy=0 1.57079632679 0 -> xyz=0 -0.153333333333 -0.32 rpy=0 1.57079632679 0
- joint drawer2_left_joint: origin xyz=-0.6825 -0.2175 0 rpy=0 0 1.57079632679 -> xyz=-0.4075 -0.145833333333 0 rpy=0 0 1.57079632679
- joint drawer2_right_joint: origin xyz=0.6825 -0.2175 0 rpy=0 0 1.57079632679 -> xyz=0.4075 -0.145833333333 0 rpy=0 0 1.57079632679
- joint drawer2_top_joint: origin xyz=0 -0.2175 0.46 rpy=1.57079632679 0 0 -> xyz=0 -0.145833333333 0.275 rpy=1.57079632679 0 0
- joint drawer3_bottom_joint: origin xyz=0 -0.2175 -0.46 rpy=1.57079632679 0 0 -> xyz=0 -0.145833333333 -0.275 rpy=1.57079632679 0 0
- joint drawer3_handle_joint: origin xyz=0 -0.23 -0.52 rpy=0 1.57079632679 0 -> xyz=0 -0.153333333333 -0.32 rpy=0 1.57079632679 0
- joint drawer3_left_joint: origin xyz=-0.6825 -0.2175 0 rpy=0 0 1.57079632679 -> xyz=-0.4075 -0.145833333333 0 rpy=0 0 1.57079632679
- joint drawer3_right_joint: origin xyz=0.6825 -0.2175 0 rpy=0 0 1.57079632679 -> xyz=0.4075 -0.145833333333 0 rpy=0 0 1.57079632679
- joint drawer3_top_joint: origin xyz=0 -0.2175 0.46 rpy=1.57079632679 0 0 -> xyz=0 -0.145833333333 0.275 rpy=1.57079632679 0 0
- joint drawer_joint1: limit lower=0.0 upper=0.8 effort=10.0 velocity=1.5 -> lower=0.0 upper=0.48 effort=10.0 velocity=1.5; origin xyz=0 -0.0275 0.0675 rpy=-1.57079632679 0 0 -> xyz=0 -0.0175 0.0425 rpy=-1.57079632679 0 0
- joint drawer_joint2: limit lower=0.0 upper=0.8 effort=10.0 velocity=1.5 -> lower=0.0 upper=0.48 effort=10.0 velocity=1.5; origin xyz=0 -0.0275 0.5325 rpy=-1.57079632679 0 0 -> xyz=0 -0.0175 0.354166666667 rpy=-1.57079632679 0 0
- joint drawer_joint3: limit lower=0.0 upper=0.8 effort=10.0 velocity=1.5 -> lower=0.0 upper=0.48 effort=10.0 velocity=1.5; origin xyz=0 -0.0275 0.9975 rpy=-1.57079632679 0 0 -> xyz=0 -0.0175 0.665833333333 rpy=-1.57079632679 0 0
- joint frame_bottom_joint: origin xyz=0 -0.475 -0.725 rpy=1.57079632679 0 0 -> xyz=0 -0.285 -0.485 rpy=1.57079632679 0 0
- joint frame_joint: origin xyz=0 0.475 0.75 rpy=0 0 0 -> xyz=0 0.285 0.5 rpy=0 0 0
- joint frame_left_joint: origin xyz=-0.725 -0.475 0 rpy=0 0 1.57079632679 -> xyz=-0.435 -0.285 0 rpy=0 0 1.57079632679
- joint frame_right_joint: origin xyz=0.725 -0.475 0 rpy=0 0 1.57079632679 -> xyz=0.435 -0.285 0 rpy=0 0 1.57079632679
- joint frame_top_joint: origin xyz=0 -0.475 0.725 rpy=1.57079632679 0 0 -> xyz=0 -0.285 0.485 rpy=1.57079632679 0 0

File: data/cupboard_drawers/cupboard_drawers.urdf.xacro (robot description, xacro)
@@ -1,10 +1,22 @@
 <?xml version="1.0" ?>
 <robot xmlns:xacro="http://www.ros.org/wiki/xacro" name="cupboard_drawers">
-<xacro:property name="wall_thickness" value="0.05"/>
-<xacro:property name="total_height" value="1.5"/>
-<xacro:property name="total_width" value="1.5"/>
-<xacro:property name="total_depth" value="1.0"/>
+<xacro:property name="wall_thickness" value="0.03"/>
+<xacro:property name="total_height" value="1.0"/>
+<xacro:property name="total_width" value="0.9"/>
+<xacro:property name="total_depth" value="0.6"/>
 <xacro:property name="num_drawers" value="3"/>
 <xacro:property name="drawer_spacing" value="0.005"/>
+<material name="white">
+  <color rgba="1 1 1 1"/>
+</material>
+<material name="dark_brown">
+  <color rgba="0.4 0.2 0.0 1"/>
+</material>
+<material name="light_brown">
+  <color rgba="0.6 0.29 0.0 1"/>
+</material>
+<material name="silver">
+  <color rgba="0.87 0.87 0.87 0.8"/>
+</material>
 <xacro:macro name="ori_geo" params="width depth height">
   <origin rpy="0 0 0" xyz="0 0 0"/>
@@ -13,5 +25,5 @@
   </geometry>
 </xacro:macro>
-<xacro:macro name="wall" params="prefix width height thickness">
+<xacro:macro name="wall" params="prefix width height thickness color">
   <link name="${prefix}_wall">
     <contact>
@@ -25,7 +37,5 @@
     <visual>
       <xacro:ori_geo width="${width}" depth="${thickness}" height="${height}"/>
-      <material name="white">
-        <color rgba="1 1 1 1"/>
-      </material>
+      <material name="${color}"/>
     </visual>
     <collision>
@@ -34,7 +44,7 @@
   </link>
 </xacro:macro>
-<xacro:macro name="corpus" params="prefix width depth height wall_thickness">
-  <xacro:wall prefix="${prefix}_back" width="${width-2*wall_thickness}" height="${height-2*wall_thickness}" thickness="${wall_thickness}"/>
-  <xacro:wall prefix="${prefix}_bottom" width="${width}" height="${depth}" thickness="${wall_thickness}"/>
+<xacro:macro name="corpus" params="prefix width depth height wall_thickness color">
+  <xacro:wall prefix="${prefix}_back" width="${width-2*wall_thickness}" height="${height-2*wall_thickness}" thickness="${wall_thickness}" color="${color}"/>
+  <xacro:wall prefix="${prefix}_bottom" width="${width}" height="${depth}" thickness="${wall_thickness}" color="${color}"/>
   <joint name="${prefix}_bottom_joint" type="fixed">
     <origin xyz="0 -${depth/2-wall_thickness/2} -${height/2-wall_thickness/2}" rpy="${pi/2} 0 0"/>
@@ -42,5 +52,5 @@
     <child link="${prefix}_bottom_wall"/>
   </joint>
-  <xacro:wall prefix="${prefix}_left" width="${depth}" height="${height-2*wall_thickness}" thickness="${wall_thickness}"/>
+  <xacro:wall prefix="${prefix}_left" width="${depth}" height="${height-2*wall_thickness}" thickness="${wall_thickness}" color="${color}"/>
   <joint name="${prefix}_left_joint" type="fixed">
     <origin xyz="-${width/2-wall_thickness/2} -${depth/2-wall_thickness/2} 0" rpy="0 0 ${pi/2}"/>
@@ -48,5 +58,5 @@
     <child link="${prefix}_left_wall"/>
   </joint>
-  <xacro:wall prefix="${prefix}_right" width="${depth}" height="${height-2*wall_thickness}" thickness="${wall_thickness}"/>
+  <xacro:wall prefix="${prefix}_right" width="${depth}" height="${height-2*wall_thickness}" thickness="${wall_thickness}" color="${color}"/>
   <joint name="${prefix}_right_joint" type="fixed">
     <origin xyz="${width/2-wall_thickness/2} -${depth/2-wall_thickness/2} 0" rpy="0 0 ${pi/2}"/>
@@ -54,5 +64,5 @@
     <child link="${prefix}_right_wall"/>
   </joint>
-  <xacro:wall prefix="${prefix}_top" width="${width}" height="${depth}" thickness="${wall_thickness}"/>
+  <xacro:wall prefix="${prefix}_top" width="${width}" height="${depth}" thickness="${wall_thickness}" color="${color}"/>
   <joint name="${prefix}_top_joint" type="fixed">
     <origin xyz="0 -${depth/2-wall_thickness/2} ${height/2-wall_thickness/2}" rpy="${pi/2} 0 0"/>
@@ -67,5 +77,6 @@
               depth="${drawer_height}"
               height="${total_depth-wall_thickness-drawer_spacing}"
-              wall_thickness="${wall_thickness*0.5}"/>
+              wall_thickness="${wall_thickness*0.5}"
+              color="light_brown"/>
   <joint name="drawer_joint${index}" type="prismatic">
     <origin xyz="0 -${(wall_thickness+drawer_spacing)/2} ${wall_thickness+drawer_spacing+0.5*0.5*wall_thickness + (index-1)*(drawer_height+drawer_spacing)}" rpy="-${pi/2} 0 0"/>
@@ -85,5 +96,5 @@
       <origin rpy="0 0 0" xyz="0 0 0"/>
       <geometry>
-        <cylinder radius="0.03" length="0.3"/>
+        <cylinder radius="0.02" length="${total_width*0.5}"/>
       </geometry>
     </collision>
@@ -91,9 +102,7 @@
       <origin rpy="0 0 0" xyz="0 0 0"/>
       <geometry>
-        <cylinder radius="0.03" length="0.3"/>
+        <cylinder radius="0.02" length="${total_width*0.5}"/>
       </geometry>
-      <material name="white">
-        <color rgba="1 1 1 1"/>
-      </material>
+      <material name="silver"/>
     </visual>
   </link>
@@ -111,5 +120,5 @@
   </inertial>
 </link>
-<xacro:corpus prefix="frame" width="${total_width}" depth="${total_depth}" height="${total_height}" wall_thickness="${wall_thickness}"/>
+<xacro:corpus prefix="frame" width="${total_width}" depth="${total_depth}" height="${total_height}" wall_thickness="${wall_thickness}" color="dark_brown"/>
 <joint name="frame_joint" type="fixed">
   <origin xyz="0 ${total_depth/2-wall_thickness/2} ${total_height/2}" rpy="0 0 0"/>

Commit message: Fixed navigation s.t. cupboard is always approached from the same direction.

File: data/cupboard_drawers/cupboard_drawers.urdf (robot description, URDF)
Before this commit: robot cupboard_drawers, 24 links, 23 joints
Links:
- added link drawer_handle_dummy_link1, mass 0.1
- added link drawer_handle_dummy_link2, mass 0.1
- added link drawer_handle_dummy_link3, mass 0.1
Joints:
- added joint drawer_handle_dummy_joint1: type fixed, parent drawer1_handle, child drawer_handle_dummy_link1, origin xyz=0 0 0 rpy=0 0 0
- added joint drawer_handle_dummy_joint2: type fixed, parent drawer2_handle, child drawer_handle_dummy_link2, origin xyz=0 0 0 rpy=0 0 0
- added joint drawer_handle_dummy_joint3: type fixed, parent drawer3_handle, child drawer_handle_dummy_link3, origin xyz=0 0 0 rpy=0 0 0

File: data/cupboard_drawers/cupboard_drawers.urdf.xacro (robot description, xacro)
@@ -112,4 +112,17 @@
     <child link="drawer${index}_handle"/>
   </joint>
+  <link name="drawer_handle_dummy_link${index}">
+    <!-- This dummy link is added s.t. the handle is the parent of some link and we can find the handle's index. -->
+    <inertial>
+      <origin rpy="0 0 0" xyz="0 0 0"/>
+      <mass value="0.1"/>
+      <inertia ixx="1" ixy="0" ixz="0" iyy="1" iyz="0" izz="1"/>
+    </inertial>
+  </link>
+  <joint name="drawer_handle_dummy_joint${index}" type="fixed">
+    <origin xyz="0 0 0" rpy="0 0 0"/>
+    <parent link="drawer${index}_handle"/>
+    <child link="drawer_handle_dummy_link${index}"/>
+  </joint>
 </xacro:macro>
 <link name="base_link">

Commit message: Robot can open drawers now

File: data/cupboard_drawers/cupboard_drawers.urdf (robot description, URDF)
Before this commit: robot cupboard_drawers, 27 links, 26 joints
Links:
- added link drawer4_back_wall, mass 0.2; collision box size=0.8 0.015 0.535; visual box size=0.8 0.015 0.535
- added link drawer4_bottom_wall, mass 0.2; collision box size=0.83 0.015 0.20375; visual box size=0.83 0.015 0.20375
- added link drawer4_handle, mass 0.2; collision cylinder length=0.36 radius=0.01; visual cylinder length=0.36 radius=0.01
- added link drawer4_left_wall, mass 0.2; collision box size=0.20375 0.015 0.535; visual box size=0.20375 0.015 0.535
- added link drawer4_right_wall, mass 0.2; collision box size=0.20375 0.015 0.535; visual box size=0.20375 0.015 0.535
- added link drawer4_top_wall, mass 0.2; collision box size=0.83 0.015 0.20375; visual box size=0.83 0.015 0.20375
- added link drawer_handle_dummy_link4, mass 0.1
- link drawer1_bottom_wall: geometry collision box size=0.83 0.015 0.20375; visual box size=0.83 0.015 0.20375
- link drawer1_handle: geometry collision cylinder length=0.36 radius=0.01; visual cylinder length=0.36 radius=0.01
- link drawer1_left_wall: geometry collision box size=0.20375 0.015 0.535; visual box size=0.20375 0.015 0.535
- link drawer1_right_wall: geometry collision box size=0.20375 0.015 0.535; visual box size=0.20375 0.015 0.535
- link drawer1_top_wall: geometry collision box size=0.83 0.015 0.20375; visual box size=0.83 0.015 0.20375
- link drawer2_bottom_wall: geometry collision box size=0.83 0.015 0.20375; visual box size=0.83 0.015 0.20375
- link drawer2_handle: geometry collision cylinder length=0.36 radius=0.01; visual cylinder length=0.36 radius=0.01
- link drawer2_left_wall: geometry collision box size=0.20375 0.015 0.535; visual box size=0.20375 0.015 0.535
- link drawer2_right_wall: geometry collision box size=0.20375 0.015 0.535; visual box size=0.20375 0.015 0.535
- link drawer2_top_wall: geometry collision box size=0.83 0.015 0.20375; visual box size=0.83 0.015 0.20375
- link drawer3_bottom_wall: geometry collision box size=0.83 0.015 0.20375; visual box size=0.83 0.015 0.20375
- link drawer3_handle: geometry collision cylinder length=0.36 radius=0.01; visual cylinder length=0.36 radius=0.01
- link drawer3_left_wall: geometry collision box size=0.20375 0.015 0.535; visual box size=0.20375 0.015 0.535
- link drawer3_right_wall: geometry collision box size=0.20375 0.015 0.535; visual box size=0.20375 0.015 0.535
- link drawer3_top_wall: geometry collision box size=0.83 0.015 0.20375; visual box size=0.83 0.015 0.20375
- link frame_back_wall: geometry collision box size=0.84 0.03 0.84; visual box size=0.84 0.03 0.84
- link frame_left_wall: geometry collision box size=0.6 0.03 0.84; visual box size=0.6 0.03 0.84
- link frame_right_wall: geometry collision box size=0.6 0.03 0.84; visual box size=0.6 0.03 0.84
Joints:
- added joint drawer4_bottom_joint: type fixed, parent drawer4_back_wall, child drawer4_bottom_wall, origin xyz=0 -0.094375 -0.275 rpy=1.57079632679 0 0
- added joint drawer4_handle_joint: type fixed, parent drawer4_back_wall, child drawer4_handle, origin xyz=0 -0.101875 -0.32 rpy=0 1.57079632679 0
- added joint drawer4_left_joint: type fixed, parent drawer4_back_wall, child drawer4_left_wall, origin xyz=-0.4075 -0.094375 0 rpy=0 0 1.57079632679
- added joint drawer4_right_joint: type fixed, parent drawer4_back_wall, child drawer4_right_wall, origin xyz=0.4075 -0.094375 0 rpy=0 0 1.57079632679
- added joint drawer4_top_joint: type fixed, parent drawer4_back_wall, child drawer4_top_wall, origin xyz=0 -0.094375 0.275 rpy=1.57079632679 0 0
- added joint drawer_handle_dummy_joint4: type fixed, parent drawer4_handle, child drawer_handle_dummy_link4, origin xyz=0 0 0 rpy=0 0 0
- added joint drawer_joint4: type prismatic, parent base_link, child drawer4_back_wall, origin xyz=0 -0.0175 0.66875 rpy=-1.57079632679 0 0, axis 0 0 -1, limit lower=0.0 upper=0.48 effort=10.0 velocity=1.5
- joint drawer1_bottom_joint: origin xyz=0 -0.145833333333 -0.275 rpy=1.57079632679 0 0 -> xyz=0 -0.094375 -0.275 rpy=1.57079632679 0 0
- joint drawer1_handle_joint: origin xyz=0 -0.153333333333 -0.32 rpy=0 1.57079632679 0 -> xyz=0 -0.101875 -0.32 rpy=0 1.57079632679 0
- joint drawer1_left_joint: origin xyz=-0.4075 -0.145833333333 0 rpy=0 0 1.57079632679 -> xyz=-0.4075 -0.094375 0 rpy=0 0 1.57079632679
- joint drawer1_right_joint: origin xyz=0.4075 -0.145833333333 0 rpy=0 0 1.57079632679 -> xyz=0.4075 -0.094375 0 rpy=0 0 1.57079632679
- joint drawer1_top_joint: origin xyz=0 -0.145833333333 0.275 rpy=1.57079632679 0 0 -> xyz=0 -0.094375 0.275 rpy=1.57079632679 0 0
- joint drawer2_bottom_joint: origin xyz=0 -0.145833333333 -0.275 rpy=1.57079632679 0 0 -> xyz=0 -0.094375 -0.275 rpy=1.57079632679 0 0
- joint drawer2_handle_joint: origin xyz=0 -0.153333333333 -0.32 rpy=0 1.57079632679 0 -> xyz=0 -0.101875 -0.32 rpy=0 1.57079632679 0
- joint drawer2_left_joint: origin xyz=-0.4075 -0.145833333333 0 rpy=0 0 1.57079632679 -> xyz=-0.4075 -0.094375 0 rpy=0 0 1.57079632679
- joint drawer2_right_joint: origin xyz=0.4075 -0.145833333333 0 rpy=0 0 1.57079632679 -> xyz=0.4075 -0.094375 0 rpy=0 0 1.57079632679
- joint drawer2_top_joint: origin xyz=0 -0.145833333333 0.275 rpy=1.57079632679 0 0 -> xyz=0 -0.094375 0.275 rpy=1.57079632679 0 0
- joint drawer3_bottom_joint: origin xyz=0 -0.145833333333 -0.275 rpy=1.57079632679 0 0 -> xyz=0 -0.094375 -0.275 rpy=1.57079632679 0 0
- joint drawer3_handle_joint: origin xyz=0 -0.153333333333 -0.32 rpy=0 1.57079632679 0 -> xyz=0 -0.101875 -0.32 rpy=0 1.57079632679 0
- joint drawer3_left_joint: origin xyz=-0.4075 -0.145833333333 0 rpy=0 0 1.57079632679 -> xyz=-0.4075 -0.094375 0 rpy=0 0 1.57079632679
- joint drawer3_right_joint: origin xyz=0.4075 -0.145833333333 0 rpy=0 0 1.57079632679 -> xyz=0.4075 -0.094375 0 rpy=0 0 1.57079632679
- joint drawer3_top_joint: origin xyz=0 -0.145833333333 0.275 rpy=1.57079632679 0 0 -> xyz=0 -0.094375 0.275 rpy=1.57079632679 0 0
- joint drawer_joint2: origin xyz=0 -0.0175 0.354166666667 rpy=-1.57079632679 0 0 -> xyz=0 -0.0175 0.25125 rpy=-1.57079632679 0 0
- joint drawer_joint3: origin xyz=0 -0.0175 0.665833333333 rpy=-1.57079632679 0 0 -> xyz=0 -0.0175 0.46 rpy=-1.57079632679 0 0
- joint frame_bottom_joint: origin xyz=0 -0.285 -0.485 rpy=1.57079632679 0 0 -> xyz=0 -0.285 -0.435 rpy=1.57079632679 0 0
- joint frame_joint: origin xyz=0 0.285 0.5 rpy=0 0 0 -> xyz=0 0.285 0.45 rpy=0 0 0
- joint frame_top_joint: origin xyz=0 -0.285 0.485 rpy=1.57079632679 0 0 -> xyz=0 -0.285 0.435 rpy=1.57079632679 0 0

File: data/cupboard_drawers/cupboard_drawers.urdf.xacro (robot description, xacro)
@@ -2,8 +2,8 @@
 <robot xmlns:xacro="http://www.ros.org/wiki/xacro" name="cupboard_drawers">
 <xacro:property name="wall_thickness" value="0.03"/>
-<xacro:property name="total_height" value="1.0"/>
+<xacro:property name="total_height" value="0.9"/>
 <xacro:property name="total_width" value="0.9"/>
 <xacro:property name="total_depth" value="0.6"/>
-<xacro:property name="num_drawers" value="3"/>
+<xacro:property name="num_drawers" value="4"/>
 <xacro:property name="drawer_spacing" value="0.005"/>
 <material name="white">
@@ -96,5 +96,5 @@
       <origin rpy="0 0 0" xyz="0 0 0"/>
       <geometry>
-        <cylinder radius="0.02" length="${total_width*0.5}"/>
+        <cylinder radius="0.01" length="${total_width*0.4}"/>
       </geometry>
     </collision>
@@ -102,5 +102,5 @@
       <origin rpy="0 0 0" xyz="0 0 0"/>
       <geometry>
-        <cylinder radius="0.02" length="${total_width*0.5}"/>
+        <cylinder radius="0.01" length="${total_width*0.4}"/>
       </geometry>
       <material name="silver"/>
@@ -142,3 +142,4 @@
 <xacro:drawer index="2"/>
 <xacro:drawer index="3"/>
+<xacro:drawer index="4"/>
 </robot>
