Commit message: Some minor modifications to make everything run more smoothly

File: data/models/box_panda_hand.urdf (robot description, URDF)
Before this commit: robot mopa, 15 links, 14 joints
Links:
- removed link realsense_link
Joints:
- removed joint camera_joint_panda_hand

Commit message: Added force sensor reading to simulated robot arm.

File: data/models/box_panda_hand.urdf (robot description, URDF)
Before this commit: robot mopa, 14 links, 13 joints
Links:
- added link panda_default_EE, mass 0.01
Joints:
- added joint joint_link8_default_ee: type fixed, parent panda_link8, child panda_default_EE, origin xyz=0.000 0.000 0.103 rpy=0.000 0.000 -0.785
