Commit message: Coloring the robot joints for a nicer look

File: data/models/box_panda_hand.urdf.xacro (robot description, xacro)
@@ -3,22 +3,4 @@
   <material name="dark_grey">
     <color rgba="0.2 0.2 0.2 1.0"/>
-  </material>
-  <material name="light_grey">
-    <color rgba="0.4 0.4 0.4 1.0"/>
-  </material>
-  <material name="red">
-    <color rgba="0.8 0.0 0.0 1.0"/>
-  </material>
-  <material name="white">
-    <color rgba="0.9 0.9 0.9 1.0"/>
-  </material>
-  <material name="yellow">
-    <color rgba="0.8 0.8 0.0 1.0"/>
-  </material>
-  <material name="black">
-    <color rgba="0.15 0.15 0.15 1.0"/>
-  </material>
-  <material name="blueish">
-    <color rgba="0.01 0.73 0.99 1.0"/>
   </material>
   <link name="base_box"/>

Commit message: Added debug error to visualize direction vector, tuned parameters a bit

File: data/models/box_panda_hand.urdf.xacro (robot description, xacro)
@@ -45,5 +45,5 @@
     <parent link="panda_link8"/>
     <child link="panda_default_EE"/>
-    <origin rpy="0.000 0.000 -0.785" xyz="0.000 0.000 0.103"/>
+    <origin rpy="0.000 0.000 ${-pi/4}" xyz="0.000 0.000 0.103"/>
   </joint>
 </robot>

File: data/models/box_panda_hand_pb.urdf (robot description, URDF)
Before this commit: robot mopa, 15 links, 14 joints
Links:
- link panda_hand: mass 0.73 -> None
- link panda_leftfinger: mass 0.1 -> None
- link panda_link0: mass 2.92 -> None
- link panda_link1: mass 2.74 -> None
- link panda_link2: mass 2.74 -> None
- link panda_link3: mass 2.38 -> None
- link panda_link4: mass 2.38 -> None
- link panda_link5: mass 2.74 -> None
- link panda_link6: mass 1.55 -> None
- link panda_link7: mass 0.54 -> None
- link panda_rightfinger: mass 0.1 -> None
Joints:
- joint joint_link8_default_ee: origin xyz=0.000 0.000 0.103 rpy=0.000 0.000 -0.785 -> xyz=0.000 0.000 0.103 rpy=0.000 0.000 -0.785398163397
