Commit message: Tuned parameters of move skill and added plotting

File: data/models/box_panda_hand_pb.urdf (robot description, URDF)
Before this commit: robot mopa, 15 links, 14 joints
Links:
- link panda_hand: mass None -> 0.73
- link panda_leftfinger: mass None -> 0.1
- link panda_link0: mass None -> 2.92
- link panda_link1: mass None -> 2.74
- link panda_link2: mass None -> 2.74
- link panda_link3: mass None -> 2.38
- link panda_link4: mass None -> 2.38
- link panda_link5: mass None -> 2.74
- link panda_link6: mass None -> 1.55
- link panda_link7: mass None -> 0.54
- link panda_rightfinger: mass None -> 0.1
