Commit message: Changed handle of cupboard to square. Made grasping handle more robust. Regenerated URDFs

File: data/models/cupboard_drawers/cupboard_drawers.urdf (robot description, URDF)
Before this commit: robot cupboard_drawers, 34 links, 33 joints
Links:
- link drawer1_handle: geometry collision box size=0.015 0.015 0.36; visual box size=0.015 0.015 0.36
- link drawer2_handle: geometry collision box size=0.015 0.015 0.36; visual box size=0.015 0.015 0.36
- link drawer3_handle: geometry collision box size=0.015 0.015 0.36; visual box size=0.015 0.015 0.36
- link drawer4_handle: geometry collision box size=0.015 0.015 0.36; visual box size=0.015 0.015 0.36

File: data/models/cupboard_drawers/cupboard_drawers.urdf.xacro (robot description, xacro)
@@ -96,5 +96,6 @@
       <origin rpy="0 0 0" xyz="0 0 0"/>
       <geometry>
-        <cylinder radius="0.01" length="${total_width*0.4}"/>
+        <!-- <cylinder radius="0.01" length="${total_width*0.4}"/> -->
+        <box size="0.015 0.015 ${total_width*0.4}"/>
       </geometry>
     </collision>
@@ -102,5 +103,6 @@
       <origin rpy="0 0 0" xyz="0 0 0"/>
       <geometry>
-        <cylinder radius="0.01" length="${total_width*0.4}"/>
+        <!-- <cylinder radius="0.01" length="${total_width*0.4}"/> -->
+        <box size="0.015 0.015 ${total_width*0.4}"/>
       </geometry>
       <material name="silver"/>

Commit message: Minor

File: data/models/cupboard_drawers/cupboard_drawers.urdf (robot description, URDF)
Before this commit: robot cupboard_drawers, 34 links, 33 joints
Links:
- link drawer1_bottom_wall: geometry collision box size=0.83 0.015 0.15375; visual box size=0.83 0.015 0.15375
- link drawer1_left_wall: geometry collision box size=0.15375 0.015 0.535; visual box size=0.15375 0.015 0.535
- link drawer1_right_wall: geometry collision box size=0.15375 0.015 0.535; visual box size=0.15375 0.015 0.535
- link drawer1_top_wall: geometry collision box size=0.83 0.015 0.15375; visual box size=0.83 0.015 0.15375
- link drawer2_bottom_wall: geometry collision box size=0.83 0.015 0.15375; visual box size=0.83 0.015 0.15375
- link drawer2_left_wall: geometry collision box size=0.15375 0.015 0.535; visual box size=0.15375 0.015 0.535
- link drawer2_right_wall: geometry collision box size=0.15375 0.015 0.535; visual box size=0.15375 0.015 0.535
- link drawer2_top_wall: geometry collision box size=0.83 0.015 0.15375; visual box size=0.83 0.015 0.15375
- link drawer3_bottom_wall: geometry collision box size=0.83 0.015 0.15375; visual box size=0.83 0.015 0.15375
- link drawer3_left_wall: geometry collision box size=0.15375 0.015 0.535; visual box size=0.15375 0.015 0.535
- link drawer3_right_wall: geometry collision box size=0.15375 0.015 0.535; visual box size=0.15375 0.015 0.535
- link drawer3_top_wall: geometry collision box size=0.83 0.015 0.15375; visual box size=0.83 0.015 0.15375
- link drawer4_bottom_wall: geometry collision box size=0.83 0.015 0.15375; visual box size=0.83 0.015 0.15375
- link drawer4_left_wall: geometry collision box size=0.15375 0.015 0.535; visual box size=0.15375 0.015 0.535
- link drawer4_right_wall: geometry collision box size=0.15375 0.015 0.535; visual box size=0.15375 0.015 0.535
- link drawer4_top_wall: geometry collision box size=0.83 0.015 0.15375; visual box size=0.83 0.015 0.15375
- link frame_back_wall: geometry collision box size=0.84 0.03 0.64; visual box size=0.84 0.03 0.64
- link frame_left_wall: geometry collision box size=0.6 0.03 0.64; visual box size=0.6 0.03 0.64
- link frame_right_wall: geometry collision box size=0.6 0.03 0.64; visual box size=0.6 0.03 0.64
Joints:
- joint drawer1_bottom_joint: origin xyz=0 -0.094375 -0.275 rpy=1.57079632679 0 0 -> xyz=0 -0.069375 -0.275 rpy=1.57079632679 0 0
- joint drawer1_handle_joint: origin xyz=0 -0.101875 -0.32 rpy=0 1.57079632679 0 -> xyz=0 -0.076875 -0.32 rpy=0 1.57079632679 0
- joint drawer1_left_joint: origin xyz=-0.4075 -0.094375 0 rpy=0 0 1.57079632679 -> xyz=-0.4075 -0.069375 0 rpy=0 0 1.57079632679
- joint drawer1_right_joint: origin xyz=0.4075 -0.094375 0 rpy=0 0 1.57079632679 -> xyz=0.4075 -0.069375 0 rpy=0 0 1.57079632679
- joint drawer1_top_joint: origin xyz=0 -0.094375 0.275 rpy=1.57079632679 0 0 -> xyz=0 -0.069375 0.275 rpy=1.57079632679 0 0
- joint drawer2_bottom_joint: origin xyz=0 -0.094375 -0.275 rpy=1.57079632679 0 0 -> xyz=0 -0.069375 -0.275 rpy=1.57079632679 0 0
- joint drawer2_handle_joint: origin xyz=0 -0.101875 -0.32 rpy=0 1.57079632679 0 -> xyz=0 -0.076875 -0.32 rpy=0 1.57079632679 0
- joint drawer2_left_joint: origin xyz=-0.4075 -0.094375 0 rpy=0 0 1.57079632679 -> xyz=-0.4075 -0.069375 0 rpy=0 0 1.57079632679
- joint drawer2_right_joint: origin xyz=0.4075 -0.094375 0 rpy=0 0 1.57079632679 -> xyz=0.4075 -0.069375 0 rpy=0 0 1.57079632679
- joint drawer2_top_joint: origin xyz=0 -0.094375 0.275 rpy=1.57079632679 0 0 -> xyz=0 -0.069375 0.275 rpy=1.57079632679 0 0
- joint drawer3_bottom_joint: origin xyz=0 -0.094375 -0.275 rpy=1.57079632679 0 0 -> xyz=0 -0.069375 -0.275 rpy=1.57079632679 0 0
- joint drawer3_handle_joint: origin xyz=0 -0.101875 -0.32 rpy=0 1.57079632679 0 -> xyz=0 -0.076875 -0.32 rpy=0 1.57079632679 0
- joint drawer3_left_joint: origin xyz=-0.4075 -0.094375 0 rpy=0 0 1.57079632679 -> xyz=-0.4075 -0.069375 0 rpy=0 0 1.57079632679
- joint drawer3_right_joint: origin xyz=0.4075 -0.094375 0 rpy=0 0 1.57079632679 -> xyz=0.4075 -0.069375 0 rpy=0 0 1.57079632679
- joint drawer3_top_joint: origin xyz=0 -0.094375 0.275 rpy=1.57079632679 0 0 -> xyz=0 -0.069375 0.275 rpy=1.57079632679 0 0
- joint drawer4_bottom_joint: origin xyz=0 -0.094375 -0.275 rpy=1.57079632679 0 0 -> xyz=0 -0.069375 -0.275 rpy=1.57079632679 0 0
- joint drawer4_handle_joint: origin xyz=0 -0.101875 -0.32 rpy=0 1.57079632679 0 -> xyz=0 -0.076875 -0.32 rpy=0 1.57079632679 0
- joint drawer4_left_joint: origin xyz=-0.4075 -0.094375 0 rpy=0 0 1.57079632679 -> xyz=-0.4075 -0.069375 0 rpy=0 0 1.57079632679
- joint drawer4_right_joint: origin xyz=0.4075 -0.094375 0 rpy=0 0 1.57079632679 -> xyz=0.4075 -0.069375 0 rpy=0 0 1.57079632679
- joint drawer4_top_joint: origin xyz=0 -0.094375 0.275 rpy=1.57079632679 0 0 -> xyz=0 -0.069375 0.275 rpy=1.57079632679 0 0
- joint drawer_joint2: origin xyz=0 -0.0175 0.25125 rpy=-1.57079632679 0 0 -> xyz=0 -0.0175 0.20125 rpy=-1.57079632679 0 0
- joint drawer_joint3: origin xyz=0 -0.0175 0.46 rpy=-1.57079632679 0 0 -> xyz=0 -0.0175 0.36 rpy=-1.57079632679 0 0
- joint drawer_joint4: origin xyz=0 -0.0175 0.66875 rpy=-1.57079632679 0 0 -> xyz=0 -0.0175 0.51875 rpy=-1.57079632679 0 0
- joint frame_bottom_joint: origin xyz=0 -0.285 -0.435 rpy=1.57079632679 0 0 -> xyz=0 -0.285 -0.335 rpy=1.57079632679 0 0
- joint frame_joint: origin xyz=0 0.285 0.45 rpy=0 0 0 -> xyz=0 0.285 0.35 rpy=0 0 0
- joint frame_top_joint: origin xyz=0 -0.285 0.435 rpy=1.57079632679 0 0 -> xyz=0 -0.285 0.335 rpy=1.57079632679 0 0

File: data/models/cupboard_drawers/cupboard_drawers.urdf.xacro (robot description, xacro)
@@ -2,5 +2,5 @@
 <robot xmlns:xacro="http://www.ros.org/wiki/xacro" name="cupboard_drawers">
 <xacro:property name="wall_thickness" value="0.03"/>
-<xacro:property name="total_height" value="0.9"/>
+<xacro:property name="total_height" value="0.7"/>
 <xacro:property name="total_width" value="0.9"/>
 <xacro:property name="total_depth" value="0.6"/>
