Commit message: Changed the way the world is created and improved URDFs

File: data/models/container/lid.urdf (robot description, URDF)
Before this commit: robot lid, 7 links, 6 joints
Joints:
- joint frame_joint: origin xyz=0 0 0.15 rpy=3.14159265359 0 0 -> xyz=0 0 0 rpy=3.14159265359 0 0

File: data/models/container/lid.urdf.xacro (robot description, xacro)
@@ -17,5 +17,5 @@
 </joint>
 <joint name="frame_joint" type="fixed">
-  <origin xyz="0 0 ${total_height+0.05}" rpy="${pi} 0 0"/>
+  <origin xyz="0 0 0" rpy="${pi} 0 0"/>
   <parent link="base_link"/>
   <child link="lid_bottom_plane"/>
