Commit message: Try to get move skill working

File: highlevel_planning/data/models/box_panda_hand.urdf.xacro (robot description, xacro)
@@ -32,5 +32,5 @@
   <xacro:include filename="$(find franka_description)/robots/panda_arm.xacro"/>
   <xacro:include filename="$(find franka_description)/robots/hand.xacro"/>
-  <xacro:panda_arm connected_to="ridgeback_dummy" xyz="0.2 0 0.45" rpy="0 0 0" />
+  <xacro:panda_arm connected_to="ridgeback_dummy" xyz="0.2 0 0.35" rpy="0 0 0" />
   <xacro:hand ns="panda" rpy="0 0 ${-pi/4}" connected_to="panda_link8"/>
   <!-- Add EE frame -->

File: highlevel_planning/data/models/box_panda_hand_pb.urdf (robot description, URDF)
Before this commit: robot mopa, 15 links, 14 joints
Joints:
- joint panda_joint_ridgeback_dummy: origin xyz=0.2 0 0.45 rpy=0 0 0 -> xyz=0.2 0 0.35 rpy=0 0 0
