Commit message: Reran xacro

File: highlevel_planning/data/models/box_panda_hand_pb.urdf (robot description, URDF)
Before this commit: robot mopa, 15 links, 14 joints
Links:
- link panda_hand: geometry collision mesh filename=/home/fjulian/Code/ros_manipulation_ws/src/moma/submodules/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; visual mesh filename=/home/fjulian/Code/ros_manipulation_ws/src/moma/submodules/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
- link panda_leftfinger: geometry collision mesh filename=/home/fjulian/Code/ros_manipulation_ws/src/moma/submodules/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; visual mesh filename=/home/fjulian/Code/ros_manipulation_ws/src/moma/submodules/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
- link panda_link0: geometry collision mesh filename=/home/fjulian/Code/ros_manipulation_ws/src/moma/submodules/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; visual mesh filename=/home/fjulian/Code/ros_manipulation_ws/src/moma/submodules/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
- link panda_link1: geometry collision mesh filename=/home/fjulian/Code/ros_manipulation_ws/src/moma/submodules/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; visual mesh filename=/home/fjulian/Code/ros_manipulation_ws/src/moma/submodules/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
- link panda_link2: geometry collision mesh filename=/home/fjulian/Code/ros_manipulation_ws/src/moma/submodules/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; visual mesh filename=/home/fjulian/Code/ros_manipulation_ws/src/moma/submodules/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
- link panda_link3: geometry collision mesh filename=/home/fjulian/Code/ros_manipulation_ws/src/moma/submodules/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; visual mesh filename=/home/fjulian/Code/ros_manipulation_ws/src/moma/submodules/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
- link panda_link4: geometry collision mesh filename=/home/fjulian/Code/ros_manipulation_ws/src/moma/submodules/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; visual mesh filename=/home/fjulian/Code/ros_manipulation_ws/src/moma/submodules/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
- link panda_link5: geometry collision mesh filename=/home/fjulian/Code/ros_manipulation_ws/src/moma/submodules/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; visual mesh filename=/home/fjulian/Code/ros_manipulation_ws/src/moma/submodules/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
- link panda_link6: geometry collision mesh filename=/home/fjulian/Code/ros_manipulation_ws/src/moma/submodules/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; visual mesh filename=/home/fjulian/Code/ros_manipulation_ws/src/moma/submodules/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
- link panda_link7: geometry collision mesh filename=/home/fjulian/Code/ros_manipulation_ws/src/moma/submodules/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; visual mesh filename=/home/fjulian/Code/ros_manipulation_ws/src/moma/submodules/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
- link panda_rightfinger: geometry collision mesh filename=/home/fjulian/Code/ros_manipulation_ws/src/moma/submodules/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; visual mesh filename=/home/fjulian/Code/ros_manipulation_ws/src/moma/submodules/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
Joints:
- joint joint_link8_default_ee: origin xyz=0.000 0.000 0.103 rpy=0.000 0.000 -0.785398163397 -> xyz=0.000 0.000 0.103 rpy=0.000 0.000 -0.7853981633974483
- joint panda_hand_joint: origin xyz=0 0 0 rpy=0 0 -0.785398163397 -> xyz=0 0 0 rpy=0 0 -0.7853981633974483
- joint panda_joint2: origin xyz=0 0 0 rpy=-1.57079632679 0 0 -> xyz=0 0 0 rpy=-1.5707963267948966 0 0
- joint panda_joint3: origin xyz=0 -0.316 0 rpy=1.57079632679 0 0 -> xyz=0 -0.316 0 rpy=1.5707963267948966 0 0
- joint panda_joint4: origin xyz=0.0825 0 0 rpy=1.57079632679 0 0 -> xyz=0.0825 0 0 rpy=1.5707963267948966 0 0
- joint panda_joint5: origin xyz=-0.0825 0.384 0 rpy=-1.57079632679 0 0 -> xyz=-0.0825 0.384 0 rpy=-1.5707963267948966 0 0
- joint panda_joint6: origin xyz=0 0 0 rpy=1.57079632679 0 0 -> xyz=0 0 0 rpy=1.5707963267948966 0 0
- joint panda_joint7: origin xyz=0.088 0 0 rpy=1.57079632679 0 0 -> xyz=0.088 0 0 rpy=1.5707963267948966 0 0

File: highlevel_planning/data/models/container/container_no_lid.urdf (robot description, URDF)
Before this commit: robot container_no_lid, 6 links, 5 joints
Links:
- link frame_back_plane: geometry collision box size=0.3 0.09000000000000001 0.01; visual box size=0.3 0.09000000000000001 0.01
- link frame_front_plane: geometry collision box size=0.3 0.09000000000000001 0.01; visual box size=0.3 0.09000000000000001 0.01
- link frame_left_plane: geometry collision box size=0.18000000000000002 0.09000000000000001 0.01; visual box size=0.18000000000000002 0.09000000000000001 0.01
- link frame_right_plane: geometry collision box size=0.18000000000000002 0.09000000000000001 0.01; visual box size=0.18000000000000002 0.09000000000000001 0.01
Joints:
- joint frame_back_joint: origin xyz=0 0.095 0.04 rpy=1.57079632679 0 0 -> xyz=0 0.095 0.04000000000000001 rpy=1.5707963267948966 0 0
- joint frame_front_joint: origin xyz=0 -0.095 0.04 rpy=1.57079632679 0 0 -> xyz=0 -0.095 0.04000000000000001 rpy=1.5707963267948966 0 0
- joint frame_left_joint: origin xyz=-0.145 0 0.04 rpy=1.57079632679 0 1.57079632679 -> xyz=-0.145 0 0.04000000000000001 rpy=1.5707963267948966 0 1.5707963267948966
- joint frame_right_joint: origin xyz=0.145 0 0.04 rpy=1.57079632679 0 1.57079632679 -> xyz=0.145 0 0.04000000000000001 rpy=1.5707963267948966 0 1.5707963267948966

File: highlevel_planning/data/models/container/container_sliding_lid.urdf (robot description, URDF)
Before this commit: robot container_no_lid, 8 links, 7 joints
Links:
- link frame_back_plane: geometry collision box size=0.3 0.09000000000000001 0.01; visual box size=0.3 0.09000000000000001 0.01
- link frame_front_plane: geometry collision box size=0.3 0.09000000000000001 0.01; visual box size=0.3 0.09000000000000001 0.01
- link frame_left_plane: geometry collision box size=0.18000000000000002 0.09000000000000001 0.01; visual box size=0.18000000000000002 0.09000000000000001 0.01
- link frame_right_plane: geometry collision box size=0.18000000000000002 0.09000000000000001 0.01; visual box size=0.18000000000000002 0.09000000000000001 0.01
- link handle: geometry collision cylinder length=0.16000000000000003 radius=0.01; visual cylinder length=0.16000000000000003 radius=0.01
- link lid_plane: geometry collision box size=0.315 0.21000000000000002 0.01; visual box size=0.315 0.21000000000000002 0.01
Joints:
- joint frame_back_joint: origin xyz=0 0.095 0.04 rpy=1.57079632679 0 0 -> xyz=0 0.095 0.04000000000000001 rpy=1.5707963267948966 0 0
- joint frame_front_joint: origin xyz=0 -0.095 0.04 rpy=1.57079632679 0 0 -> xyz=0 -0.095 0.04000000000000001 rpy=1.5707963267948966 0 0
- joint frame_left_joint: origin xyz=-0.145 0 0.04 rpy=1.57079632679 0 1.57079632679 -> xyz=-0.145 0 0.04000000000000001 rpy=1.5707963267948966 0 1.5707963267948966
- joint frame_right_joint: origin xyz=0.145 0 0.04 rpy=1.57079632679 0 1.57079632679 -> xyz=0.145 0 0.04000000000000001 rpy=1.5707963267948966 0 1.5707963267948966
- joint handle_joint: origin xyz=0 0 0.025 rpy=1.57079632679 0 0 -> xyz=0 0 0.025 rpy=1.5707963267948966 0 0
- joint lid_joint: origin xyz=0 0 0.09 rpy=0 0 0 -> xyz=0 0 0.09000000000000001 rpy=0 0 0

File: highlevel_planning/data/models/container/lid.urdf (robot description, URDF)
Before this commit: robot lid, 7 links, 6 joints
Links:
- link lid_back_plane: geometry collision box size=0.33999999999999997 0.020000000000000004 0.01; visual box size=0.33999999999999997 0.020000000000000004 0.01
- link lid_bottom_plane: geometry collision box size=0.33999999999999997 0.24000000000000002 0.01; visual box size=0.33999999999999997 0.24000000000000002 0.01
- link lid_front_plane: geometry collision box size=0.33999999999999997 0.020000000000000004 0.01; visual box size=0.33999999999999997 0.020000000000000004 0.01
- link lid_left_plane: geometry collision box size=0.22000000000000003 0.020000000000000004 0.01; visual box size=0.22000000000000003 0.020000000000000004 0.01
- link lid_right_plane: geometry collision box size=0.22000000000000003 0.020000000000000004 0.01; visual box size=0.22000000000000003 0.020000000000000004 0.01
Joints:
- joint frame_joint: origin xyz=0 0 0 rpy=3.14159265359 0 0 -> xyz=0 0 0 rpy=3.141592653589793 0 0
- joint handle_joint: origin xyz=0 0 -0.025 rpy=0 1.57079632679 0 -> xyz=0 0 -0.025 rpy=0 1.5707963267948966 0
- joint lid_back_joint: origin xyz=0 0.115 0.005 rpy=1.57079632679 0 0 -> xyz=0 0.115 0.005000000000000002 rpy=1.5707963267948966 0 0
- joint lid_front_joint: origin xyz=0 -0.115 0.005 rpy=1.57079632679 0 0 -> xyz=0 -0.115 0.005000000000000002 rpy=1.5707963267948966 0 0
- joint lid_left_joint: origin xyz=-0.165 0 0.005 rpy=1.57079632679 0 1.57079632679 -> xyz=-0.16499999999999998 0 0.005000000000000002 rpy=1.5707963267948966 0 1.5707963267948966
- joint lid_right_joint: origin xyz=0.165 0 0.005 rpy=1.57079632679 0 1.57079632679 -> xyz=0.16499999999999998 0 0.005000000000000002 rpy=1.5707963267948966 0 1.5707963267948966

File: highlevel_planning/data/models/cupboard_drawers/cupboard_drawers.urdf (robot description, URDF)
Before this commit: robot cupboard_drawers, 34 links, 33 joints
Links:
- link drawer1_back_wall: geometry collision box size=0.8 0.015 0.5349999999999999; visual box size=0.8 0.015 0.5349999999999999
- link drawer1_bottom_wall: geometry collision box size=0.8300000000000001 0.015 0.15374999999999997; visual box size=0.8300000000000001 0.015 0.15374999999999997
- link drawer1_handle: geometry collision box size=0.015 0.015 0.36000000000000004; visual box size=0.015 0.015 0.36000000000000004
- link drawer1_left_wall: geometry collision box size=0.15374999999999997 0.015 0.5349999999999999; visual box size=0.15374999999999997 0.015 0.5349999999999999
- link drawer1_right_wall: geometry collision box size=0.15374999999999997 0.015 0.5349999999999999; visual box size=0.15374999999999997 0.015 0.5349999999999999
- link drawer1_top_wall: geometry collision box size=0.8300000000000001 0.015 0.15374999999999997; visual box size=0.8300000000000001 0.015 0.15374999999999997
- link drawer2_back_wall: geometry collision box size=0.8 0.015 0.5349999999999999; visual box size=0.8 0.015 0.5349999999999999
- link drawer2_bottom_wall: geometry collision box size=0.8300000000000001 0.015 0.15374999999999997; visual box size=0.8300000000000001 0.015 0.15374999999999997
- link drawer2_handle: geometry collision box size=0.015 0.015 0.36000000000000004; visual box size=0.015 0.015 0.36000000000000004
- link drawer2_left_wall: geometry collision box size=0.15374999999999997 0.015 0.5349999999999999; visual box size=0.15374999999999997 0.015 0.5349999999999999
- link drawer2_right_wall: geometry collision box size=0.15374999999999997 0.015 0.5349999999999999; visual box size=0.15374999999999997 0.015 0.5349999999999999
- link drawer2_top_wall: geometry collision box size=0.8300000000000001 0.015 0.15374999999999997; visual box size=0.8300000000000001 0.015 0.15374999999999997
- link drawer3_back_wall: geometry collision box size=0.8 0.015 0.5349999999999999; visual box size=0.8 0.015 0.5349999999999999
- link drawer3_bottom_wall: geometry collision box size=0.8300000000000001 0.015 0.15374999999999997; visual box size=0.8300000000000001 0.015 0.15374999999999997
- link drawer3_handle: geometry collision box size=0.015 0.015 0.36000000000000004; visual box size=0.015 0.015 0.36000000000000004
- link drawer3_left_wall: geometry collision box size=0.15374999999999997 0.015 0.5349999999999999; visual box size=0.15374999999999997 0.015 0.5349999999999999
- link drawer3_right_wall: geometry collision box size=0.15374999999999997 0.015 0.5349999999999999; visual box size=0.15374999999999997 0.015 0.5349999999999999
- link drawer3_top_wall: geometry collision box size=0.8300000000000001 0.015 0.15374999999999997; visual box size=0.8300000000000001 0.015 0.15374999999999997
- link drawer4_back_wall: geometry collision box size=0.8 0.015 0.5349999999999999; visual box size=0.8 0.015 0.5349999999999999
- link drawer4_bottom_wall: geometry collision box size=0.8300000000000001 0.015 0.15374999999999997; visual box size=0.8300000000000001 0.015 0.15374999999999997
- link drawer4_handle: geometry collision box size=0.015 0.015 0.36000000000000004; visual box size=0.015 0.015 0.36000000000000004
- link drawer4_left_wall: geometry collision box size=0.15374999999999997 0.015 0.5349999999999999; visual box size=0.15374999999999997 0.015 0.5349999999999999
- link drawer4_right_wall: geometry collision box size=0.15374999999999997 0.015 0.5349999999999999; visual box size=0.15374999999999997 0.015 0.5349999999999999
- link drawer4_top_wall: geometry collision box size=0.8300000000000001 0.015 0.15374999999999997; visual box size=0.8300000000000001 0.015 0.15374999999999997
- link frame_back_wall: geometry collision box size=0.8400000000000001 0.03 0.6399999999999999; visual box size=0.8400000000000001 0.03 0.6399999999999999
- link frame_left_wall: geometry collision box size=0.6 0.03 0.6399999999999999; visual box size=0.6 0.03 0.6399999999999999
- link frame_right_wall: geometry collision box size=0.6 0.03 0.6399999999999999; visual box size=0.6 0.03 0.6399999999999999
Joints:
- joint drawer1_bottom_joint: origin xyz=0 -0.069375 -0.275 rpy=1.57079632679 0 0 -> xyz=0 -0.06937499999999999 -0.27499999999999997 rpy=1.5707963267948966 0 0
- joint drawer1_handle_joint: origin xyz=0 -0.076875 -0.32 rpy=0 1.57079632679 0 -> xyz=0 -0.07687499999999999 -0.32 rpy=0 1.5707963267948966 0
- joint drawer1_left_joint: origin xyz=-0.4075 -0.069375 0 rpy=0 0 1.57079632679 -> xyz=-0.40750000000000003 -0.06937499999999999 0 rpy=0 0 1.5707963267948966
- joint drawer1_right_joint: origin xyz=0.4075 -0.069375 0 rpy=0 0 1.57079632679 -> xyz=0.40750000000000003 -0.06937499999999999 0 rpy=0 0 1.5707963267948966
- joint drawer1_top_joint: origin xyz=0 -0.069375 0.275 rpy=1.57079632679 0 0 -> xyz=0 -0.06937499999999999 0.27499999999999997 rpy=1.5707963267948966 0 0
- joint drawer2_bottom_joint: origin xyz=0 -0.069375 -0.275 rpy=1.57079632679 0 0 -> xyz=0 -0.06937499999999999 -0.27499999999999997 rpy=1.5707963267948966 0 0
- joint drawer2_handle_joint: origin xyz=0 -0.076875 -0.32 rpy=0 1.57079632679 0 -> xyz=0 -0.07687499999999999 -0.32 rpy=0 1.5707963267948966 0
- joint drawer2_left_joint: origin xyz=-0.4075 -0.069375 0 rpy=0 0 1.57079632679 -> xyz=-0.40750000000000003 -0.06937499999999999 0 rpy=0 0 1.5707963267948966
- joint drawer2_right_joint: origin xyz=0.4075 -0.069375 0 rpy=0 0 1.57079632679 -> xyz=0.40750000000000003 -0.06937499999999999 0 rpy=0 0 1.5707963267948966
- joint drawer2_top_joint: origin xyz=0 -0.069375 0.275 rpy=1.57079632679 0 0 -> xyz=0 -0.06937499999999999 0.27499999999999997 rpy=1.5707963267948966 0 0
- joint drawer3_bottom_joint: origin xyz=0 -0.069375 -0.275 rpy=1.57079632679 0 0 -> xyz=0 -0.06937499999999999 -0.27499999999999997 rpy=1.5707963267948966 0 0
- joint drawer3_handle_joint: origin xyz=0 -0.076875 -0.32 rpy=0 1.57079632679 0 -> xyz=0 -0.07687499999999999 -0.32 rpy=0 1.5707963267948966 0
- joint drawer3_left_joint: origin xyz=-0.4075 -0.069375 0 rpy=0 0 1.57079632679 -> xyz=-0.40750000000000003 -0.06937499999999999 0 rpy=0 0 1.5707963267948966
- joint drawer3_right_joint: origin xyz=0.4075 -0.069375 0 rpy=0 0 1.57079632679 -> xyz=0.40750000000000003 -0.06937499999999999 0 rpy=0 0 1.5707963267948966
- joint drawer3_top_joint: origin xyz=0 -0.069375 0.275 rpy=1.57079632679 0 0 -> xyz=0 -0.06937499999999999 0.27499999999999997 rpy=1.5707963267948966 0 0
- joint drawer4_bottom_joint: origin xyz=0 -0.069375 -0.275 rpy=1.57079632679 0 0 -> xyz=0 -0.06937499999999999 -0.27499999999999997 rpy=1.5707963267948966 0 0
- joint drawer4_handle_joint: origin xyz=0 -0.076875 -0.32 rpy=0 1.57079632679 0 -> xyz=0 -0.07687499999999999 -0.32 rpy=0 1.5707963267948966 0
- joint drawer4_left_joint: origin xyz=-0.4075 -0.069375 0 rpy=0 0 1.57079632679 -> xyz=-0.40750000000000003 -0.06937499999999999 0 rpy=0 0 1.5707963267948966
- joint drawer4_right_joint: origin xyz=0.4075 -0.069375 0 rpy=0 0 1.57079632679 -> xyz=0.40750000000000003 -0.06937499999999999 0 rpy=0 0 1.5707963267948966
- joint drawer4_top_joint: origin xyz=0 -0.069375 0.275 rpy=1.57079632679 0 0 -> xyz=0 -0.06937499999999999 0.27499999999999997 rpy=1.5707963267948966 0 0
- joint drawer_joint1: origin xyz=0 -0.0175 0.0425 rpy=-1.57079632679 0 0 -> xyz=0 -0.017499999999999998 0.042499999999999996 rpy=-1.5707963267948966 0 0
- joint drawer_joint2: origin xyz=0 -0.0175 0.20125 rpy=-1.57079632679 0 0 -> xyz=0 -0.017499999999999998 0.20124999999999998 rpy=-1.5707963267948966 0 0
- joint drawer_joint3: origin xyz=0 -0.0175 0.36 rpy=-1.57079632679 0 0 -> xyz=0 -0.017499999999999998 0.35999999999999993 rpy=-1.5707963267948966 0 0
- joint drawer_joint4: origin xyz=0 -0.0175 0.51875 rpy=-1.57079632679 0 0 -> xyz=0 -0.017499999999999998 0.5187499999999999 rpy=-1.5707963267948966 0 0
- joint frame_bottom_joint: origin xyz=0 -0.285 -0.335 rpy=1.57079632679 0 0 -> xyz=0 -0.285 -0.33499999999999996 rpy=1.5707963267948966 0 0
- joint frame_left_joint: origin xyz=-0.435 -0.285 0 rpy=0 0 1.57079632679 -> xyz=-0.435 -0.285 0 rpy=0 0 1.5707963267948966
- joint frame_right_joint: origin xyz=0.435 -0.285 0 rpy=0 0 1.57079632679 -> xyz=0.435 -0.285 0 rpy=0 0 1.5707963267948966
- joint frame_top_joint: origin xyz=0 -0.285 0.335 rpy=1.57079632679 0 0 -> xyz=0 -0.285 0.33499999999999996 rpy=1.5707963267948966 0 0

Commit message: Adopted latest version of franka description

File: highlevel_planning/data/models/box_panda_hand_pb.urdf (robot description, URDF)
Before this commit: robot mopa, 15 links, 14 joints
Links:
- link panda_hand: geometry collision cylinder length=0.1 radius=0.04; collision sphere radius=0.04
- link panda_link0: geometry collision cylinder length=0.03 radius=0.06; collision sphere radius=0.06
- link panda_link1: geometry collision cylinder length=0.2830 radius=0.06; collision sphere radius=0.06
- link panda_link2: geometry collision cylinder length=0.12 radius=0.06; collision sphere radius=0.06
- link panda_link3: geometry collision cylinder length=0.15 radius=0.06; collision sphere radius=0.06
- link panda_link4: geometry collision cylinder length=0.12 radius=0.06; collision sphere radius=0.06
- link panda_link5: geometry collision cylinder length=0.1 radius=0.06; collision cylinder length=0.14 radius=0.025
- link panda_link6: geometry collision cylinder length=0.08 radius=0.05; collision sphere radius=0.05
- link panda_link7: geometry collision cylinder length=0.14 radius=0.04; collision sphere radius=0.04
Joints:
- joint panda_joint8: axis 0 0 0 -> (none)

Commit message: Updated URDFs

File: highlevel_planning/data/models/box_panda_hand_pb.urdf (robot description, URDF)
Before this commit: robot mopa, 15 links, 14 joints
Links:
- link panda_hand: mass 0.73 -> 0.68
- link panda_leftfinger: mass 0.1 -> 0.68
- link panda_link0: mass 2.92 -> 3.06
- link panda_link1: mass 2.74 -> 2.34; geometry collision mesh filename=/home/fjulian/Code/ros_manipulation_ws/src/moma/submodules/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; visual mesh filename=/home/fjulian/Code/ros_manipulation_ws/src/moma/submodules/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
- link panda_link2: mass 2.74 -> 2.36
- link panda_link4: mass 2.38 -> 2.43
- link panda_link5: mass 2.74 -> 3.5
- link panda_link6: mass 1.55 -> 1.47
- link panda_link7: mass 0.54 -> 0.45
- link panda_link8: mass None -> 0.45
- link panda_rightfinger: mass 0.1 -> 0.68

File: highlevel_planning/data/models/cupboard2/cupboard2.urdf (robot description, URDF)
Before this commit: robot cupboard_drawers, 6 links, 5 joints
Links:
- link corpus_link: geometry collision mesh filename=/home/fjulian/Code/ros_manipulation_ws/src/asl_highlevel_pl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; visual mesh filename=/home/fjulian/Code/ros_manipulation_ws/src/asl_highlevel_pl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
- link drawer1_link: geometry collision mesh filename=/home/fjulian/Code/ros_manipulation_ws/src/asl_highlevel_pl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; visual mesh filename=/home/fjulian/Code/ros_manipulation_ws/src/asl_highlevel_pl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
- link drawer2_link: geometry collision mesh filename=/home/fjulian/Code/ros_manipulation_ws/src/asl_highlevel_pl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; visual mesh filename=/home/fjulian/Code/ros_manipulation_ws/src/asl_highlevel_pl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
- link drawer3_link: geometry collision mesh filename=/home/fjulian/Code/ros_manipulation_ws/src/asl_highlevel_pl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; visual mesh filename=/home/fjulian/Code/ros_manipulation_ws/src/asl_highlevel_pl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
- link drawer4_link: geometry collision mesh filename=/home/fjulian/Code/ros_manipulation_ws/src/asl_highlevel_pl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; visual mesh filename=/home/fjulian/Code/ros_manipulation_ws/src/asl_highlevel_pl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
