Commit message: Added shelf URDF

File: highlevel_planning/data/models/common.xacro (robot description, xacro)
@@ -1,9 +1,4 @@
 <?xml version="1.0"?>
 <robot xmlns:xacro="http://www.ros.org/wiki/xacro" name="container_common">
-<xacro:property name="wall_thickness" value="0.01"/>
-<xacro:property name="total_height" value="0.1"/>
-<xacro:property name="total_width" value="0.3"/>
-<xacro:property name="total_depth" value="0.2"/>
-<xacro:property name="lid_spacing" value="0.01"/>
 <material name="white">
   <color rgba="1 1 1 1"/>

File: highlevel_planning/data/models/container/container_no_lid.urdf.xacro (robot description, xacro)
@@ -1,5 +1,10 @@
 <?xml version="1.0"?>
 <robot xmlns:xacro="http://www.ros.org/wiki/xacro" name="container_no_lid">
-<xacro:include filename="container_common.xacro"/>
+<xacro:include filename="$(cwd)/common.xacro"/>
+<xacro:property name="wall_thickness" value="0.01"/>
+<xacro:property name="total_height" value="0.1"/>
+<xacro:property name="total_width" value="0.3"/>
+<xacro:property name="total_depth" value="0.2"/>
+<xacro:property name="lid_spacing" value="0.01"/>
 <link name="base_link">
   <inertial>

File: highlevel_planning/data/models/container/container_sliding_lid.urdf.xacro (robot description, xacro)
@@ -1,5 +1,10 @@
 <?xml version="1.0"?>
 <robot xmlns:xacro="http://www.ros.org/wiki/xacro" name="container_no_lid">
-<xacro:include filename="container_common.xacro"/>
+<xacro:include filename="$(cwd)/common.xacro"/>
+<xacro:property name="wall_thickness" value="0.01"/>
+<xacro:property name="total_height" value="0.1"/>
+<xacro:property name="total_width" value="0.3"/>
+<xacro:property name="total_depth" value="0.2"/>
+<xacro:property name="lid_spacing" value="0.01"/>
 <link name="base_link">
   <inertial>

File: highlevel_planning/data/models/container/lid.urdf.xacro (robot description, xacro)
@@ -1,5 +1,10 @@
 <?xml version="1.0"?>
 <robot xmlns:xacro="http://www.ros.org/wiki/xacro" name="lid">
-<xacro:include filename="container_common.xacro"/>
+<xacro:include filename="$(cwd)/common.xacro"/>
+<xacro:property name="wall_thickness" value="0.01"/>
+<xacro:property name="total_height" value="0.1"/>
+<xacro:property name="total_width" value="0.3"/>
+<xacro:property name="total_depth" value="0.2"/>
+<xacro:property name="lid_spacing" value="0.01"/>
 <link name="base_link">
   <inertial>

File: highlevel_planning/data/models/cupboard2/cupboard2.urdf.xacro (robot description, xacro)
@@ -32,5 +32,5 @@
                 <origin rpy="0 0 0" xyz="0 0 0"/>
                 <geometry>
-                    <mesh filename="$(find highlevel_planning)/data/models/cupboard2/corpus.stl"/>
+                    <mesh filename="$(find highlevel_planning_ros1)/../../highlevel_planning/data/models/cupboard2/corpus.stl"/>
                 </geometry>
             </collision>
@@ -38,5 +38,5 @@
                 <origin rpy="0 0 0" xyz="0 0 0"/>
                 <geometry>
-                    <mesh filename="$(find highlevel_planning)/data/models/cupboard2/corpus.stl"/>
+                    <mesh filename="$(find highlevel_planning_ros1)/../../highlevel_planning/data/models/cupboard2/corpus.stl"/>
                 </geometry>
                 <material name="dark_brown"/>
@@ -57,5 +57,5 @@
                 <origin rpy="0 0 0" xyz="0 0 0"/>
                 <geometry>
-                    <mesh filename="$(find highlevel_planning)/data/models/cupboard2/drawer.stl"/>
+                    <mesh filename="$(find highlevel_planning_ros1)/../../highlevel_planning/data/models/cupboard2/drawer.stl"/>
                 </geometry>
             </collision>
@@ -63,5 +63,5 @@
                 <origin rpy="0 0 0" xyz="0 0 0"/>
                 <geometry>
-                    <mesh filename="$(find highlevel_planning)/data/models/cupboard2/drawer.stl"/>
+                    <mesh filename="$(find highlevel_planning_ros1)/../../highlevel_planning/data/models/cupboard2/drawer.stl"/>
                 </geometry>
                 <material name="light_brown"/>
