Commit message: Added coke can

File: highlevel_planning/data/models/shelf/shelf.urdf (robot description, URDF)
Before this commit: robot container_no_lid, 8 links, 7 joints
Links:
- link board0_plane: geometry collision box size=0.25 0.6699999999999999 0.03; visual box size=0.25 0.6699999999999999 0.03
- link board1_plane: geometry collision box size=0.25 0.6699999999999999 0.03; visual box size=0.25 0.6699999999999999 0.03
- link board2_plane: geometry collision box size=0.25 0.6699999999999999 0.03; visual box size=0.25 0.6699999999999999 0.03
- link board3_plane: geometry collision box size=0.25 0.6699999999999999 0.03; visual box size=0.25 0.6699999999999999 0.03
- link board4_plane: geometry collision box size=0.25 0.6699999999999999 0.03; visual box size=0.25 0.6699999999999999 0.03
- link left_wall_plane: geometry collision box size=0.25 0.8 0.03; visual box size=0.25 0.8 0.03
- link right_wall_plane: geometry collision box size=0.25 0.8 0.03; visual box size=0.25 0.8 0.03
Joints:
- joint board1_joint: origin xyz=0 0 0.3075 rpy=0 0 0 -> xyz=0 0 0.20750000000000002 rpy=0 0 0
- joint board2_joint: origin xyz=0 0 0.6 rpy=0 0 0 -> xyz=0 0 0.4 rpy=0 0 0
- joint board3_joint: origin xyz=0 0 0.8925 rpy=0 0 0 -> xyz=0 0 0.5925 rpy=0 0 0
- joint board4_joint: origin xyz=0 0 1.1849999999999998 rpy=0 0 0 -> xyz=0 0 0.785 rpy=0 0 0
- joint left_wall_joint: origin xyz=0 -0.65 0.6 rpy=1.5707963267948966 0 0 -> xyz=0 -0.35 0.4 rpy=1.5707963267948966 0 0
- joint right_wall_joint: origin xyz=0 0.65 0.6 rpy=1.5707963267948966 0 0 -> xyz=0 0.35 0.4 rpy=1.5707963267948966 0 0

File: highlevel_planning/data/models/shelf/shelf.urdf.xacro (robot description, xacro)
@@ -2,7 +2,7 @@
 <robot xmlns:xacro="http://www.ros.org/wiki/xacro" name="container_no_lid">
     <xacro:include filename="$(cwd)/common.xacro"/>
-    <xacro:property name="total_width" value="1.3"/>
-    <xacro:property name="total_height" value="1.2"/>
-    <xacro:property name="total_depth" value="0.3"/>
+    <xacro:property name="total_width" value="0.7"/>
+    <xacro:property name="total_height" value="0.8"/>
+    <xacro:property name="total_depth" value="0.25"/>
     <xacro:property name="wall_thickness" value="0.03"/>
     <xacro:property name="num_boards" value="5"/>

Commit message: Manually designed placing in shelf works

File: highlevel_planning/data/models/shelf/shelf.urdf (robot description, URDF)
Before this commit: robot container_no_lid, 8 links, 7 joints
Links:
- added link board5_plane, mass 0.2; collision box size=0.25 1.17 0.03; visual box size=0.25 1.17 0.03
- link board0_plane: geometry collision box size=0.25 1.17 0.03; visual box size=0.25 1.17 0.03
- link board1_plane: geometry collision box size=0.25 1.17 0.03; visual box size=0.25 1.17 0.03
- link board2_plane: geometry collision box size=0.25 1.17 0.03; visual box size=0.25 1.17 0.03
- link board3_plane: geometry collision box size=0.25 1.17 0.03; visual box size=0.25 1.17 0.03
- link board4_plane: geometry collision box size=0.25 1.17 0.03; visual box size=0.25 1.17 0.03
- link left_wall_plane: geometry collision box size=0.25 1.4 0.03; visual box size=0.25 1.4 0.03
- link right_wall_plane: geometry collision box size=0.25 1.4 0.03; visual box size=0.25 1.4 0.03
Joints:
- added joint board5_joint: type fixed, parent base_link, child board5_plane, origin xyz=0 0 1.3849999999999998 rpy=0 0 0
- joint board1_joint: origin xyz=0 0 0.20750000000000002 rpy=0 0 0 -> xyz=0 0 0.289 rpy=0 0 0
- joint board2_joint: origin xyz=0 0 0.4 rpy=0 0 0 -> xyz=0 0 0.563 rpy=0 0 0
- joint board3_joint: origin xyz=0 0 0.5925 rpy=0 0 0 -> xyz=0 0 0.8369999999999999 rpy=0 0 0
- joint board4_joint: origin xyz=0 0 0.785 rpy=0 0 0 -> xyz=0 0 1.1109999999999998 rpy=0 0 0
- joint left_wall_joint: origin xyz=0 -0.35 0.4 rpy=1.5707963267948966 0 0 -> xyz=0 -0.6 0.7 rpy=1.5707963267948966 0 0
- joint right_wall_joint: origin xyz=0 0.35 0.4 rpy=1.5707963267948966 0 0 -> xyz=0 0.6 0.7 rpy=1.5707963267948966 0 0

File: highlevel_planning/data/models/shelf/shelf.urdf.xacro (robot description, xacro)
@@ -2,9 +2,9 @@
 <robot xmlns:xacro="http://www.ros.org/wiki/xacro" name="container_no_lid">
     <xacro:include filename="$(cwd)/common.xacro"/>
-    <xacro:property name="total_width" value="0.7"/>
-    <xacro:property name="total_height" value="0.8"/>
+    <xacro:property name="total_width" value="1.2"/>
+    <xacro:property name="total_height" value="1.4"/>
     <xacro:property name="total_depth" value="0.25"/>
     <xacro:property name="wall_thickness" value="0.03"/>
-    <xacro:property name="num_boards" value="5"/>
+    <xacro:property name="num_boards" value="6"/>
     <link name="base_link">
         <inertial>
@@ -40,3 +40,5 @@
     <xacro:board index="3"/>
     <xacro:board index="4"/>
+    <xacro:board index="5"/>
+<!--    <xacro:board index="6"/>-->
 </robot>
